File: TLAUX/Kicad/TLAUX_Adapter_PSOC5/TLAUX_Adapter_PSOC5.kicad_pcb (KiCad board)
At the start: 2 copper layers, 28.6 x 37.5 mm, 17 parts, among them J1 USB_micro-B, P1 CONN_01X05, U2 MC68HC811E2, U3 CY8C58LP_QFN68

Commit message: had some problems with the tool changer changed the tool changer state machine to run at 1ms tweaked a lot of time constants and added a little sensor debounce.
Other:
- net class Default removed
